File: card/apple2idiot_new/apple2idiot_new.sch (KiCad schematic (older format))
At the start: 9 parts, among them J1 AppleIIBus, J2 Conn_02x02_Odd_Even, J3 Conn_01x04, J4 Conn_02x02_Odd_Even, J5 Conn_02x02_Odd_Even, J6 Conn_02x07_Odd_Even, U1 IDT7132, U2 ESP32-DEVKITC-32D

Commit message: Cleaned up rot13 example, and misc catchup from laptop
Parts:
- J1: symbol kicad-library:AppleIIBus -> apple2idiot_new-rescue:AppleIIBus-kicad-library
- U2: symbol ESP32-DEV_KIT:ESP32-DEVKITC-32D -> apple2idiot_new-rescue:ESP32-DEVKITC-32D-ESP32-DEV_KIT
Changed lines of the file:
@@
 $EndDescr
 $Comp
-L kicad-library:AppleIIBus J1
+L apple2idiot_new-rescue:AppleIIBus-kicad-library J1
 U 1 1 61291E51
 P 3400 6800
@@
 $EndComp
 $Comp
-L ESP32-DEV_KIT:ESP32-DEVKITC-32D U2
+L apple2idiot_new-rescue:ESP32-DEVKITC-32D-ESP32-DEV_KIT U2
 U 1 1 612B5485
 P 13000 5550
@@
 Text Label 9400 5950 0    50   ~ 0
 AR7
-Wire Bus Line
-	9700 5350 9700 5650
-Wire Bus Line
-	11200 5650 11200 7550
-Wire Bus Line
-	14650 4100 14650 5250
-Wire Bus Line
-	4350 5650 4350 6350
-Wire Bus Line
-	14650 5450 14650 7550
-Wire Bus Line
-	7300 6350 7300 7050
-Wire Bus Line
-	9700 6550 9700 7550
-Wire Bus Line
-	7300 4950 7300 6150
-Wire Bus Line
-	2400 4950 2400 6400
 Text Label 7500 4950 0    50   ~ 0
 BSYL
@@
 Text Label 3450 3800 0    50   ~ 0
 CEL
+Wire Bus Line
+	9700 5350 9700 5650
+Wire Bus Line
+	11200 5650 11200 7550
+Wire Bus Line
+	14650 4100 14650 5250
+Wire Bus Line
+	4350 5650 4350 6350
+Wire Bus Line
+	14650 5450 14650 7550
+Wire Bus Line
+	7300 6350 7300 7050
+Wire Bus Line
+	9700 6550 9700 7550
+Wire Bus Line
+	7300 4950 7300 6150
+Wire Bus Line
+	2400 4950 2400 6400
 $EndSCHEMATC
